File: aio3 PCB guide/_autosave-aio3 PCB guide.sch (KiCad schematic (older format))
At the start: 24 parts, among them SW1 SW_Push, U1 ATmega32U4-AU, Y1 16mhz

Commit message: DRC complete (kinda)
Parts:
- USB1: symbol random-keyboard-parts:Molex-0548190589 -> random-keyboard-parts:Molex-0548190519
Changed lines of the file:
@@
 D-
-$Comp
-L random-keyboard-parts:Molex-0548190589 USB1
-U 1 1 601012E0
-P 7100 2300
-F 0 "USB1" V 7637 2267 60  0000 C CNN
-F 1 "Molex-0548190589" V 7531 2267 60  0000 C CNN
-F 2 "random-keyboard-parts:Molex-0548190589" H 7100 2300 60  0001 C CNN
-F 3 "" H 7100 2300 60  0001 C CNN
-	1    7100 2300
-	0    -1   -1   0
-$EndComp
 $Comp
 L power:VCC #PWR0111
@@
 Text GLabel 4900 2550 2    50   Input ~ 0
 COL1
+$Comp
+L random-keyboard-parts:Molex-0548190519 USB1
+U 1 1 601012E0
+P 7100 2300
+F 0 "USB1" V 7637 2267 60  0000 C CNN
+F 1 "Molex-0548190589" V 7531 2267 60  0000 C CNN
+F 2 "random-keyboard-parts:Molex-0548190589" H 7100 2300 60  0001 C CNN
+F 3 "" H 7100 2300 60  0001 C CNN
+	1    7100 2300
+	0    -1   -1   0
+$EndComp
 $EndSCHEMATC
