File: aio3 PCB guide/aio3 PCB guide.kicad_pcb (KiCad board)
At the start: 2 copper layers, 80.2 x 38.1 mm, 24 parts, among them SW1 SW_Push, U1 ATmega32U4-AU, Y1 16mhz

Commit message: Stuff done
Parts:
- moved C1 9.05 mm to (108.7, 52.5), turned to 270 degrees
- moved C2 9.05 mm to (100.8, 52.5), turned to 90 degrees
- turned Y1 to 180 degrees
Routing:
- net GND: track 0.00 -> 25.1 mm
- net Net-(R3-Pad1): track 0.00 -> 22.6 mm
- net Net-(R2-Pad1): track 0.00 -> 20.1 mm
- net D+: track 0.00 -> 7.48 mm
- net D-: track 0.00 -> 6.50 mm
- net Net-(C2-Pad2): track 0.00 -> 2.89 mm
Changed lines of the file:
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@@
     (thickness 1.6)
     (drawings 8)
-    (tracks 0)
+    (tracks 30)
     (zones 0)
     (modules 24)
@@
   )
   (module Crystal:Crystal_SMD_3225-4Pin_3.2x2.5mm (layer B.Cu)
-    (at 104.775 52.3875)
+    (at 104.775 52.3875 180)
     (descr "SMD Crystal SERIES SMD3225/4 http://www.txccrystal.com/images/pdf/7m-accuracy.pdf, 3.2x2.5mm^2 package")
     (tags "SMD SMT crystal")
@@
       (effects (font (size 0.7 0.7) (thickness 0.105)) (justify mirror))
     )
-    (pad 4 smd rect (at -1.1 0.85) (size 1.4 1.2) (layers B.Cu B.Paste B.Mask)
-      (net 2 GND))
-    (pad 3 smd rect (at 1.1 0.85) (size 1.4 1.2) (layers B.Cu B.Paste B.Mask)
+    (pad 4 smd rect (at -1.1 0.85 180) (size 1.4 1.2) (layers B.Cu B.Paste B.Mask)
+      (net 2 GND))
+    (pad 3 smd rect (at 1.1 0.85 180) (size 1.4 1.2) (layers B.Cu B.Paste B.Mask)
       (net 3 "Net-(C2-Pad2)"))
-    (pad 2 smd rect (at 1.1 -0.85) (size 1.4 1.2) (layers B.Cu B.Paste B.Mask)
-      (net 2 GND))
-    (pad 1 smd rect (at -1.1 -0.85) (size 1.4 1.2) (layers B.Cu B.Paste B.Mask)
+    (pad 2 smd rect (at 1.1 -0.85 180) (size 1.4 1.2) (layers B.Cu B.Paste B.Mask)
+      (net 2 GND))
+    (pad 1 smd rect (at -1.1 -0.85 180) (size 1.4 1.2) (layers B.Cu B.Paste B.Mask)
       (net 1 "Net-(C1-Pad2)"))
     (model ${KISYS3DMOD}/Crystal.3dshapes/Crystal_SMD_3225-4Pin_3.2x2.5mm.wrl
@@
   )
   (module Capacitor_SMD:C_0805_2012Metric (layer B.Cu)
-    (at 109.855 52.3875)
+    (at 100.80625 52.54375 90)
     (descr "Capacitor SMD 0805 (2012 Metric), square (rectangular) end terminal, IPC_7351 nominal, (Body size source: IPC-SM-782 page 76, https://www.pcb-3d.com/wordpress/wp-content/uploads/ipc-sm-782a_amendment_1_and_2.pdf, https://docs.google.com/spreadsheets/d/1BsfQQcO9C6DZCsRaXUlFlo91Tg2WpOkGARC1WS5S8t0/edit?usp=sharing), generated with kicad-footprint-generator")
     (tags capacitor)
     (attr smd)
-    (fp_text reference C2 (at 0 1.68) (layer B.SilkS)
-      (effects (font (size 1 1) (thickness 0.15)) (justify mirror))
-    )
-    (fp_text value 22pf (at 0 -1.68) (layer B.Fab)
-      (effects (font (size 1 1) (thickness 0.15)) (justify mirror))
-    )
-    (fp_text user %R (at 0 0) (layer B.Fab)
+    (fp_text reference C2 (at 0 1.68 90) (layer B.SilkS)
+      (effects (font (size 1 1) (thickness 0.15)) (justify mirror))
+    )
+    (fp_text value 22pf (at 0 -1.68 90) (layer B.Fab)
+      (effects (font (size 1 1) (thickness 0.15)) (justify mirror))
+    )
+    (fp_text user %R (at 0 0 90) (layer B.Fab)
       (effects (font (size 0.5 0.5) (thickness 0.08)) (justify mirror))
     )
@@
     (fp_line (start -1 0.625) (end 1 0.625) (layer B.Fab) (width 0.1))
     (fp_line (start -1 -0.625) (end -1 0.625) (layer B.Fab) (width 0.1))
-    (pad 2 smd roundrect (at 0.95 0) (size 1 1.45) (layers B.Cu B.Paste B.Mask) (roundrect_rratio 0.25)
+    (pad 2 smd roundrect (at 0.95 0 90) (size 1 1.45) (layers B.Cu B.Paste B.Mask) (roundrect_rratio 0.25)
       (net 3 "Net-(C2-Pad2)"))
-    (pad 1 smd roundrect (at -0.95 0) (size 1 1.45) (layers B.Cu B.Paste B.Mask) (roundrect_rratio 0.25)
+    (pad 1 smd roundrect (at -0.95 0 90) (size 1 1.45) (layers B.Cu B.Paste B.Mask) (roundrect_rratio 0.25)
       (net 2 GND))
     (model ${KISYS3DMOD}/Capacitor_SMD.3dshapes/C_0805_2012Metric.wrl
@@
   )
   (module Capacitor_SMD:C_0805_2012Metric (layer B.Cu)
-    (at 99.695 52.3875)
+    (at 108.74375 52.54375 270)
     (descr "Capacitor SMD 0805 (2012 Metric), square (rectangular) end terminal, IPC_7351 nominal, (Body size source: IPC-SM-782 page 76, https://www.pcb-3d.com/wordpress/wp-content/uploads/ipc-sm-782a_amendment_1_and_2.pdf, https://docs.google.com/spreadsheets/d/1BsfQQcO9C6DZCsRaXUlFlo91Tg2WpOkGARC1WS5S8t0/edit?usp=sharing), generated with kicad-footprint-generator")
     (tags capacitor)
     (attr smd)
-    (fp_text reference C1 (at 0 1.68) (layer B.SilkS)
-      (effects (font (size 1 1) (thickness 0.15)) (justify mirror))
-    )
-    (fp_text value 22pf (at 0 -1.68) (layer B.Fab)
-      (effects (font (size 1 1) (thickness 0.15)) (justify mirror))
-    )
-    (fp_text user %R (at 0 0) (layer B.Fab)
+    (fp_text reference C1 (at 0 1.68 90) (layer B.SilkS)
+      (effects (font (size 1 1) (thickness 0.15)) (justify mirror))
+    )
+    (fp_text value 22pf (at 0 -1.68 90) (layer B.Fab)
+      (effects (font (size 1 1) (thickness 0.15)) (justify mirror))
+    )
+    (fp_text user %R (at 0 0 90) (layer B.Fab)
       (effects (font (size 0.5 0.5) (thickness 0.08)) (justify mirror))
     )
@@
     (fp_line (start -1 0.625) (end 1 0.625) (layer B.Fab) (width 0.1))
     (fp_line (start -1 -0.625) (end -1 0.625) (layer B.Fab) (width 0.1))
-    (pad 2 smd roundrect (at 0.95 0) (size 1 1.45) (layers B.Cu B.Paste B.Mask) (roundrect_rratio 0.25)
+    (pad 2 smd roundrect (at 0.95 0 270) (size 1 1.45) (layers B.Cu B.Paste B.Mask) (roundrect_rratio 0.25)
       (net 1 "Net-(C1-Pad2)"))
-    (pad 1 smd roundrect (at -0.95 0) (size 1 1.45) (layers B.Cu B.Paste B.Mask) (roundrect_rratio 0.25)
+    (pad 1 smd roundrect (at -0.95 0 270) (size 1 1.45) (layers B.Cu B.Paste B.Mask) (roundrect_rratio 0.25)
       (net 2 GND))
     (model ${KISYS3DMOD}/Capacitor_SMD.3dshapes/C_0805_2012Metric.wrl
@@
   (gr_arc (start 152.4 80.16875) (end 152.4 82.55) (angle -90) (layer Edge.Cuts) (width 0.05))
   (gr_arc (start 152.4 46.83125) (end 154.78125 46.83125) (angle -90) (layer Edge.Cuts) (width 0.05))
+  (segment (start 100.80625 54.09375) (end 100.80625 53.49375) (width 0.254) (layer B.Cu) (net 2))
+  (segment (start 100.80625 55.056816) (end 100.80625 54.09375) (width 0.254) (layer B.Cu) (net 2))
+  (segment (start 103.175 57.425566) (end 100.80625 55.056816) (width 0.254) (layer B.Cu) (net 2))
+  (segment (start 103.175 59.3875) (end 103.175 57.425566) (width 0.254) (layer B.Cu) (net 2))
+  (segment (start 100.80625 53.49375) (end 99.53125 53.49375) (width 0.254) (layer B.Cu) (net 2))
+  (segment (start 99.53125 53.49375) (end 99.21875 53.18125) (width 0.254) (layer B.Cu) (net 2))
+  (segment (start 105.875 50.3125) (end 105.875 51.5375) (width 0.254) (layer B.Cu) (net 2))
+  (segment (start 105.56875 50.00625) (end 105.875 50.3125) (width 0.254) (layer B.Cu) (net 2))
+  (segment (start 99.21875 50.8) (end 100.0125 50.00625) (width 0.254) (layer B.Cu) (net 2))
+  (segment (start 100.0125 50.00625) (end 105.56875 50.00625) (width 0.254) (layer B.Cu) (net 2))
+  (segment (start 99.21875 53.18125) (end 99.21875 50.8) (width 0.254) (layer B.Cu) (net 2))
+  (segment (start 108.6875 51.5375) (end 108.74375 51.59375) (width 0.254) (layer B.Cu) (net 2))
+  (segment (start 105.875 51.5375) (end 108.6875 51.5375) (width 0.254) (layer B.Cu) (net 2))
+  (segment (start 103.775 53.2375) (end 103.675 53.2375) (width 0.254) (layer B.Cu) (net 2))
+  (segment (start 105.475 51.5375) (end 103.775 53.2375) (width 0.254) (layer B.Cu) (net 2))
+  (segment (start 105.875 51.5375) (end 105.475 51.5375) (width 0.254) (layer B.Cu) (net 2))
+  (segment (start 103.61875 51.59375) (end 103.675 51.5375) (width 0.254) (layer B.Cu) (net 3))
+  (segment (start 100.80625 51.59375) (end 103.61875 51.59375) (width 0.254) (layer B.Cu) (net 3))
+  (segment (start 82.55 54.65) (end 84.93125 57.03125) (width 0.254) (layer B.Cu) (net 16))
+  (segment (start 82.55 50.5375) (end 82.55 54.65) (width 0.254) (layer B.Cu) (net 16))
+  (segment (start 88.11875 66.6875) (end 99.075 66.6875) (width 0.254) (layer B.Cu) (net 17))
+  (segment (start 84.93125 63.5) (end 88.11875 66.6875) (width 0.254) (layer B.Cu) (net 17))
+  (segment (start 84.93125 58.85625) (end 84.93125 63.5) (width 0.254) (layer B.Cu) (net 17))
+  (segment (start 81.75 57.025) (end 81.75625 57.03125) (width 0.254) (layer B.Cu) (net 18))
+  (segment (start 81.75 50.5375) (end 81.75 57.025) (width 0.254) (layer B.Cu) (net 18))
+  (segment (start 87.482933 67.4875) (end 99.075 67.4875) (width 0.254) (layer B.Cu) (net 19))
+  (segment (start 84.1375 64.142067) (end 87.482933 67.4875) (width 0.254) (layer B.Cu) (net 19))
+  (segment (start 84.1375 61.9125) (end 84.1375 64.142067) (width 0.254) (layer B.Cu) (net 19))
+  (segment (start 81.75625 58.85625) (end 81.75625 59.53125) (width 0.254) (layer B.Cu) (net 19))
+  (segment (start 81.75625 59.53125) (end 84.1375 61.9125) (width 0.254) (layer B.Cu) (net 19))
 )

Commit message: PCB routed
Parts:
- moved C7 6.12 mm to (95.4, 70.8), turned to 270 degrees
- moved R4 1.71 mm to (113.5, 70.0)
- moved C3 0.79 mm to (94.6, 64.3), turned to 180 degrees
- moved C4 0.79 mm to (95.9, 57.9)
- moved R1 0.79 mm to (92.1, 57.9), turned to 270 degrees
- turned C6 to 180 degrees
- turned F1 to 270 degrees
Routing:
- net GND: track 25.1 -> 143.8 mm
- net +5V: track 0.00 -> 98.0 mm, vias 0 -> 5
- net Net-(R1-Pad2): track 0.00 -> 35.8 mm, vias 0 -> 2
- net VCC: track 0.00 -> 13.4 mm
- net Net-(C1-Pad2): track 0.00 -> 9.58 mm
- net Net-(C2-Pad2): track 2.89 -> 12.0 mm
- net Net-(C3-Pad1): track 0.00 -> 3.84 mm
- net Net-(R4-Pad2): track 0.00 -> 3.04 mm

Commit message: Finished PCB
Parts:
- moved MX2 26.9 mm to (145.3, 54.0)
- moved MX3 26.9 mm to (126.2, 73.0)
- moved R3 1.59 mm to (80.2, 57.9)
- moved R2 0.79 mm to (84.1, 57.9)
- renumbered MX3 to MX2, MX2 to MX3
Connections:
- U1 pad 27: Net-(U1-Pad27) -> ROW0
- U1 pad 28: Net-(U1-Pad28) -> COL1
- U1 pad 29: Net-(U1-Pad29) -> COL0
- U1 pad 30: Net-(U1-Pad30) -> ROW1
Routing:
- net COL1: track 0.00 -> 52.6 mm
- net ROW1: track 0.00 -> 51.3 mm
- net ROW0: track 0.00 -> 48.5 mm
- net COL0: track 0.00 -> 33.2 mm
- net Net-(D1-Pad2): track 0.00 -> 7.44 mm
- net +5V: track 98.0 -> 104.7 mm
- net Net-(D2-Pad2): track 0.00 -> 6.62 mm
- net Net-(D4-Pad2): track 0.00 -> 6.62 mm
- net Net-(D3-Pad2): track 0.00 -> 6.62 mm
- net Net-(R2-Pad1): track 20.1 -> 24.1 mm
- net Net-(R3-Pad1): track 22.6 -> 25.3 mm
- net D-: track 6.50 -> 7.16 mm

Commit message: DRC complete (kinda)
Routing:
- added copper zone on B.Cu, net GND
Other:
- outline, holes or cut-outs redrawn
