File: aio3 PCB guide/aio3 PCB guide.sch (KiCad schematic (older format))
At the start: 25 parts, among them SW1 SW_Push, U1 ATmega32U4-AU, Y1 16mhz

Commit message: Physical layout down
Parts:
- removed MX5: MX-NoLED, MX_Alps_Hybrid:MX-1U-NoLED, symbol MX_Alps_Hybrid:MX-NoLED
- MX1, MX2, MX3, MX4: footprint MX_Alps_Hybrid:MX-1U-NoLED -> MX_Alps_Hybrid:MX-1U
Connections:
- net COL0: no longer MX4.1 (COL)
- net COL1: now also MX4.1 (COL)
- net at D1.2 (A), MX1.2 (ROW): no longer MX2.2 (ROW)
- net at D3.2 (A): now also MX2.2 (ROW); no longer MX4.2 (ROW)
- net at D4.2 (A): now also MX4.2 (ROW)
Other:
- moved on the sheet: MX2, MX4
Changed lines of the file:
@@
 EESchema Schematic File Version 4
+LIBS:aio3 PCB guide-cache
 EELAYER 30 0
 EELAYER END
@@
 F 0 "MX1" H 7283 4523 60  0000 C CNN
 F 1 "MX-NoLED" H 7283 4449 20  0000 C CNN
-F 2 "MX_Alps_Hybrid:MX-1U-NoLED" H 6625 4275 60  0001 C CNN
+F 2 "MX_Alps_Hybrid:MX-1U" H 6625 4275 60  0001 C CNN
 F 3 "" H 6625 4275 60  0001 C CNN
 	1    7250 4300
@@
 L MX_Alps_Hybrid:MX-NoLED MX2
 U 1 1 60119803
-P 7250 4300
-F 0 "MX2" H 7283 4523 60  0000 C CNN
-F 1 "MX-NoLED" H 7283 4449 20  0000 C CNN
-F 2 "MX_Alps_Hybrid:MX-1U-NoLED" H 6625 4275 60  0001 C CNN
-F 3 "" H 6625 4275 60  0001 C CNN
-	1    7250 4300
+P 7250 5050
+F 0 "MX2" H 7283 5273 60  0000 C CNN
+F 1 "MX-NoLED" H 7283 5199 20  0000 C CNN
+F 2 "MX_Alps_Hybrid:MX-1U" H 6625 5025 60  0001 C CNN
+F 3 "" H 6625 5025 60  0001 C CNN
+	1    7250 5050
 	1    0    0    -1
 $EndComp
@@
 F 0 "MX3" H 7833 4523 60  0000 C CNN
 F 1 "MX-NoLED" H 7833 4449 20  0000 C CNN
-F 2 "MX_Alps_Hybrid:MX-1U-NoLED" H 7175 4275 60  0001 C CNN
+F 2 "MX_Alps_Hybrid:MX-1U" H 7175 4275 60  0001 C CNN
 F 3 "" H 7175 4275 60  0001 C CNN
 	1    7800 4300
@@
 L MX_Alps_Hybrid:MX-NoLED MX4
 U 1 1 60120150
-P 7250 5050
-F 0 "MX4" H 7283 5273 60  0000 C CNN
-F 1 "MX-NoLED" H 7283 5199 20  0000 C CNN
-F 2 "MX_Alps_Hybrid:MX-1U-NoLED" H 6625 5025 60  0001 C CNN
-F 3 "" H 6625 5025 60  0001 C CNN
-	1    7250 5050
-	1    0    0    -1
-$EndComp
-$Comp
-L MX_Alps_Hybrid:MX-NoLED MX5
-U 1 1 60120DFE
 P 7800 5050
-F 0 "MX5" H 7833 5273 60  0000 C CNN
+F 0 "MX4" H 7833 5273 60  0000 C CNN
 F 1 "MX-NoLED" H 7833 5199 20  0000 C CNN
-F 2 "MX_Alps_Hybrid:MX-1U-NoLED" H 7175 5025 60  0001 C CNN
+F 2 "MX_Alps_Hybrid:MX-1U" H 7175 5025 60  0001 C CNN
 F 3 "" H 7175 5025 60  0001 C CNN
 	1    7800 5050
@@
 	0    -1   -1   0
 $EndComp
-Connection ~ 7200 4450
 Wire Wire Line
 	7400 5000 7400 4250

Commit message: Finished PCB
Parts:
- renumbered MX3 to MX2, MX2 to MX3
Connections:
- net COL0: now also U1.29 (PB5)
- net COL1: now also U1.28 (PB4)
- net ROW0: now also U1.27 (PD7)
- net ROW1: now also U1.30 (PB6)
Changed lines of the file:
@@
 	7100 4450 7200 4450
 $Comp
-L MX_Alps_Hybrid:MX-NoLED MX2
+L MX_Alps_Hybrid:MX-NoLED MX3
 U 1 1 60119803
 P 7250 5050
-F 0 "MX2" H 7283 5273 60  0000 C CNN
+F 0 "MX3" H 7283 5273 60  0000 C CNN
 F 1 "MX-NoLED" H 7283 5199 20  0000 C CNN
 F 2 "MX_Alps_Hybrid:MX-1U" H 6625 5025 60  0001 C CNN
@@
 $EndComp
 $Comp
-L MX_Alps_Hybrid:MX-NoLED MX3
+L MX_Alps_Hybrid:MX-NoLED MX2
 U 1 1 6011F1F5
 P 7800 4300
-F 0 "MX3" H 7833 4523 60  0000 C CNN
+F 0 "MX2" H 7833 4523 60  0000 C CNN
 F 1 "MX-NoLED" H 7833 4449 20  0000 C CNN
 F 2 "MX_Alps_Hybrid:MX-1U" H 7175 4275 60  0001 C CNN
@@
 Text GLabel 6800 4650 0    50   Input ~ 0
 ROW0
+Text GLabel 4900 4050 2    50   Input ~ 0
+ROW0
+Text GLabel 4900 2750 2    50   Input ~ 0
+ROW1
+Text GLabel 4900 2650 2    50   Input ~ 0
+COL0
+Text GLabel 4900 2550 2    50   Input ~ 0
+COL1
 $EndSCHEMATC

Commit message: DRC complete (kinda)
Parts:
- removed USB1: Molex-0548190589, random-keyboard-parts:Molex-0548190589, symbol random-keyboard-parts:Molex-0548190589
- added USB1: Molex-0548190519, random-keyboard-parts:Molex-0548190519, symbol random-keyboard-parts:Molex-0548190519
Connections:
- net D+: now also USB1.4 (D-)
- net D-: now also USB1.5 (VBUS)
- net GND: now also USB1.2 (ID)
- net VCC: now also USB1.6 (SHIELD)
Changed lines of the file:
@@
 D-
-$Comp
-L random-keyboard-parts:Molex-0548190589 USB1
-U 1 1 601012E0
-P 7100 2300
-F 0 "USB1" V 7637 2267 60  0000 C CNN
-F 1 "Molex-0548190589" V 7531 2267 60  0000 C CNN
-F 2 "random-keyboard-parts:Molex-0548190589" H 7100 2300 60  0001 C CNN
-F 3 "" H 7100 2300 60  0001 C CNN
-	1    7100 2300
-	0    -1   -1   0
-$EndComp
 $Comp
 L power:VCC #PWR0111
@@
 Text GLabel 4900 2550 2    50   Input ~ 0
 COL1
+$Comp
+L random-keyboard-parts:Molex-0548190519 USB1
+U 1 1 600F1D81
+P 7100 2400
+F 0 "USB1" V 7637 2367 60  0000 C CNN
+F 1 "Molex-0548190519" V 7531 2367 60  0000 C CNN
+F 2 "random-keyboard-parts:Molex-0548190519" H 7100 2400 60  0001 C CNN
+F 3 "" H 7100 2400 60  0001 C CNN
+	1    7100 2400
+	0    -1   -1   0
+$EndComp
 $EndSCHEMATC
